Commit message: add Turtle robot model and controller

File: urdf/Turtle.urdf (robot description, URDF)
Before this commit: robot niitblue_turtle, 4 links, 3 joints
Links:
- removed link WHEEL_L
- removed link WHEEL_R
- added link WHEEL_L0; visual cylinder length=0.018 radius=0.033
- added link WHEEL_R0; visual cylinder length=0.018 radius=0.033
Joints:
- removed joint base_link_to_WHEEL_L
- removed joint base_link_to_WHEEL_R
- added joint WHEEL_L: type continuous, parent base_link, child WHEEL_L0, origin xyz=0.033 0.08 -0.048 rpy=1.57 0 0
- added joint WHEEL_R: type continuous, parent base_link, child WHEEL_R0, origin xyz=0.033 -0.08 -0.048 rpy=-1.57 0 0
